Commit message: add lrmate200id7l  to fanuc_lrmate200id_support

File: fanuc_lrmate200id_support/urdf/lrmate200id7l_macro.xacro (robot description, xacro)
@@ -2,5 +2,5 @@
 <robot xmlns:xacro="http://www.ros.org/wiki/xacro">
   <xacro:include filename="$(find fanuc_lrmate200id_support)/urdf/common_materials.xacro"/>
-  <xacro:macro name="fanuc_lrmate200id" params="prefix">
+  <xacro:macro name="fanuc_lrmate200id7l" params="prefix">
     <!-- links: main serial chain -->
     <link name="${prefix}base_link">
@@ -52,12 +52,12 @@
         <origin xyz="0 0 0" rpy="0 0 0"/>
         <geometry>
-          <mesh filename="package://fanuc_lrmate200id_support/meshes/lrmate200id/visual/link_2.stl"/>
-        </geometry>
-        <xacro:material_fanuc_yellow />
-      </visual>
-      <collision>
-        <origin xyz="0 0 0" rpy="0 0 0"/>
-        <geometry>
-          <mesh filename="package://fanuc_lrmate200id_support/meshes/lrmate200id/collision/link_2.stl"/>
+          <mesh filename="package://fanuc_lrmate200id_support/meshes/lrmate200id7l/visual/link_2.stl" scale="0.001 0.001 0.001"/>
+        </geometry>
+        <xacro:material_fanuc_yellow />
+      </visual>
+      <collision>
+        <origin xyz="0 0 0" rpy="0 0 0"/>
+        <geometry>
+          <mesh filename="package://fanuc_lrmate200id_support/meshes/lrmate200id7l/collision/link_2.stl" scale="0.001 0.001 0.001"/>
         </geometry>
       </collision>
@@ -96,12 +96,12 @@
         <origin xyz="0 0 0" rpy="0 0 0"/>
         <geometry>
-          <mesh filename="package://fanuc_lrmate200id_support/meshes/lrmate200id/visual/link_4.stl"/>
-        </geometry>
-        <xacro:material_fanuc_yellow />
-      </visual>
-      <collision>
-        <origin xyz="0 0 0" rpy="0 0 0"/>
-        <geometry>
-          <mesh filename="package://fanuc_lrmate200id_support/meshes/lrmate200id/collision/link_4.stl"/>
+          <mesh filename="package://fanuc_lrmate200id_support/meshes/lrmate200id7l/visual/link_4.stl" scale="0.001 0.001 0.001"/>
+        </geometry>
+        <xacro:material_fanuc_yellow />
+      </visual>
+      <collision>
+        <origin xyz="0 0 0" rpy="0 0 0"/>
+        <geometry>
+          <mesh filename="package://fanuc_lrmate200id_support/meshes/lrmate200id7l/collision/link_4.stl" scale="0.001 0.001 0.001"/>
         </geometry>
       </collision>
@@ -165,7 +165,6 @@
       <axis xyz="0 0 1" />
       <limit effort="0" lower="-2.965" upper="2.965" velocity="7.85" />
-      <dynamics damping="0.0" friction="0.0"/>
-   </joint>
-   <joint name="${prefix}joint_2" type="revolute">
+    </joint>
+    <joint name="${prefix}joint_2" type="revolute">
       <origin xyz="0.050 0 0" rpy="0 0 0"/>
       <parent link="${prefix}link_1" />
@@ -175,5 +174,5 @@
     </joint>
     <joint name="${prefix}joint_3" type="revolute">
-      <origin xyz="0 0 0.330" rpy="0 0 0"/>
+      <origin xyz="0 0 0.440" rpy="0 0 0"/>
       <parent link="${prefix}link_2" />
       <child link="${prefix}link_3" />
@@ -189,5 +188,5 @@
     </joint>
     <joint name="${prefix}joint_5" type="revolute">
-      <origin xyz="0.335 0 0" rpy="0 0 0"/>
+      <origin xyz="0.420 0 0" rpy="0 0 0"/>
       <parent link="${prefix}link_4"/>
       <child link="${prefix}link_5"/>
@@ -216,9 +215,22 @@
       <child link="${prefix}flange" />
     </joint>
-    <!-- ROS-Industrial 'tool0' frame: all-zeros tool frame -->
-    <link name="${prefix}tool0" />
+    <link name="${prefix}tool0">
+      <visual>
+        <origin xyz="0 0 0" rpy="0 0 0"/>
+        <geometry>
+          <mesh filename="package://fanuc_lrmate200id_support/meshes/lrmate200id/visual/link_6.stl"/>
+        </geometry>
+        <xacro:material_fanuc_black />
+      </visual>
+      <collision>
+        <origin xyz="0 0 0" rpy="0 0 0"/>
+        <geometry>
+          <mesh filename="package://fanuc_lrmate200id_support/meshes/lrmate200id/collision/link_6.stl"/>
+        </geometry>
+      </collision>
+    </link>
     <joint name="${prefix}link_6-tool0" type="fixed">
       <origin xyz="0 0 0" rpy="${pi} ${-pi/2.0} 0" />
-      <parent link="${prefix}flange" />
+      <parent link="${prefix}link_6" />
       <child link="${prefix}tool0" />
     </joint>
