Commit message: attach cam to link_6, and calibrate it

File: fanuc_lrmate200id_support/urdf/lrmate200id7l.xacro (robot description, xacro)
@@ -5,8 +5,8 @@
        <!-- Part 6 Gripper Base Joint -->
 <joint name="camera_joint" type="fixed">
-    <parent link="link_4" />
+    <parent link="link_6" />
     <child link="camera_link" />
-    <origin rpy="-0.0037 1.50600 -0.0031"
-     xyz="0.32273 0.01841 -0.06556" />
+    <origin rpy="-0.1232 -0.0023 -0.0105"
+     xyz="0.03352 0.02587 0.06753" />
     <axis xyz="0 0 0" />
 </joint>

Commit message: reda calibration param from YAML

File: fanuc_lrmate200id_support/urdf/lrmate200id7l.xacro (robot description, xacro)
@@ -3,12 +3,3 @@
   <xacro:include filename="$(find fanuc_lrmate200id_support)/urdf/lrmate200id7l_macro.xacro"/>
   <xacro:fanuc_lrmate200id7l prefix=""/>
-       <!-- Part 6 Gripper Base Joint -->
-<joint name="camera_joint" type="fixed">
-    <parent link="link_6" />
-    <child link="camera_link" />
-    <origin rpy="-0.1232 -0.0023 -0.0105"
-     xyz="0.03352 0.02587 0.06753" />
-    <axis xyz="0 0 0" />
-</joint>
-<link name="camera_link"/>
 </robot>
