Commit message: add new gripper

File: fanuc_lrmate200id_support/urdf/gripper_macro.xacro (robot description, xacro)
@@ -3,24 +3,21 @@
 <xacro:macro name="gripper" params="prefix">
     <!-- Part 6 Gripper Base Joint -->
-    <joint name="Part6_Gripper_Base" type="revolute">
+    <joint name="gripper_base_to_link_6" type="fixed">
         <parent link="link_6" />
-        <child link="Gripper_Base" />
-        <origin rpy="0 -1.57 0" xyz="0 0 0" />
-        <axis xyz="0 0 1" />
-        <dynamics damping="0.7" />
-        <limit effort="100" lower="-0.5232" upper="0.5232" velocity="100" />
+        <child link="gripper_base_link" />
+        <origin rpy="0 0 0" xyz="0.05 0 0.0" />
     </joint>
     <!-- Gripper Base -->
-    <link name="Gripper_Base">
+    <link name="gripper_base_link">
         <collision>
-            <origin rpy="-1.57 0 0" xyz="-0.065 -0.065 0" />
+            <origin rpy="0 0 0" xyz="0 0 0" />
             <geometry>
-                <mesh filename="package://fanuc_lrmate200id_support/meshes/gripper/collision/Gripper_base.STL" scale="0.001 0.001 0.001" />
+                <mesh filename="package://fanuc_lrmate200id_support/meshes/gripper/collision/gripper_base.stl" scale="0.001 0.001 0.001" />
             </geometry>
         </collision>
         <visual>
-            <origin rpy="-1.57 0 0" xyz="-0.065 -0.065 0" />
+            <origin rpy="0 0 0" xyz="0 0 0" />
             <geometry>
-                <mesh filename="package://fanuc_lrmate200id_support/meshes/gripper/visual/Gripper_base.STL" scale="0.001 0.001 0.001" />
+                <mesh filename="package://fanuc_lrmate200id_support/meshes/gripper/visual/gripper_base.stl" scale="0.001 0.001 0.001" />
             </geometry>
             <material name="">
@@ -28,5 +25,5 @@
             </material>
         </visual>
-<inertial>
+        <inertial>
             <origin rpy="0 0 0" xyz="0.00112 0.04196 0" />
             <mass value="1.067" />
@@ -34,144 +31,105 @@
         </inertial>
     </link>
-    <gazebo reference="Gripper_Base">
+    <gazebo reference="gripper_base_link">
         <material>Gazebo/Black</material>
     </gazebo>
-    <!-- Gripper Base Finger 3 Joint-->
-    <joint name="Gripper_Finger3" type="revolute">
-        <parent link="Gripper_Base" />
-        <child link="Finger3" />
-        <origin rpy="0 0 0" xyz="0.04448 0 -0.09533" />
-        <axis xyz="0 1 0" />
-        <dynamics damping="0.7" />
-        <limit effort="1" lower="-0.0872" upper="0.0872" velocity="6.1087" />
+        <!-- Part 6 Gripper Base Joint -->
+    <joint name="mid_layer_to_gripper_base" type="fixed">
+        <parent link="gripper_base_link" />
+        <child link="mid_layer_link" />
+        <origin rpy="0 0 0" xyz="0.07 0 0.0" />
     </joint>
-    <!-- Finger 3-->
-    <link name="Finger3">
+    <!-- Gripper Base -->
+    <link name="mid_layer_link">
         <collision>
-            <origin rpy="-1.57 0 3.14" xyz="0.075 0.038 0.075" />
+            <origin rpy="0 0 0" xyz="0 0 0" />
             <geometry>
-                <mesh filename="package://fanuc_lrmate200id_support/meshes/gripper/collision/Gripper_finger.STL" scale="0.001 0.001 0.001" />
+                <mesh filename="package://fanuc_lrmate200id_support/meshes/gripper/collision/mid_layer.stl" scale="0.001 0.001 0.001" />
             </geometry>
         </collision>
         <visual>
-            <origin rpy="-1.57 0 3.14" xyz="0.075 0.038 0.075" />
+            <origin rpy="0 0 0" xyz="0 0 0" />
             <geometry>
-                <mesh filename="package://fanuc_lrmate200id_support/meshes/gripper/visual/Gripper_finger.STL" scale="0.001 0.001 0.001" />
+                <mesh filename="package://fanuc_lrmate200id_support/meshes/gripper/visual/mid_layer.stl" scale="0.001 0.001 0.001" />
             </geometry>
             <material name="">
-                <color rgba="0.278431372549 0.278431372549 0.278431372549 1.0" />
+                <color rgba="0.1 0.4 0.13 1.0" />
             </material>
         </visual>
-<inertial>
+        <inertial>
             <origin rpy="0 0 0" xyz="0.00112 0.04196 0" />
-            <mass value="0.17495" />
-            <inertia ixx="0.002449587" ixy="-0.00141880714" ixz="-0.00044070839" iyy=".00018834795" iyz="-0.00067806067" izz=".00315304482" />
+            <mass value="1.067" />
+            <inertia ixx="0.00372062398" ixy="-0.000013337910" ixz="0.000000013" iyy=".00223540544" iyz="-0.00000003496" izz=".003641916" />
         </inertial>
     </link>
-    <!-- Base Finger1 Joint -->
-    <!-- Gripper Base Finger 1 Joint-->
-    <joint name="Gripper_Finger1" type="revolute">
-        <parent link="Gripper_Base" />
-        <child link="Finger1" />
-        <origin rpy="0 0 0" xyz="-0.04448 0.04 -0.09533" />
-        <axis xyz="0 1 0" />
-        <dynamics damping="0.7" />
-        <limit effort="1" lower="-0.0872" upper="0.0872" velocity="6.1087" />
+    <gazebo reference="mid_layer_link">
+        <material>Gazebo/Black</material>
+    </gazebo>
+            <!-- Part 6 Gripper Base Joint -->
+    <joint name="finger_1_to_mid_layer" type="prismatic">
+        <parent link="mid_layer_link" />
+        <child link="finger_1_link" />
+        <origin rpy="3.14 0 0" xyz="0.10 0.032 0.0" />
+        <limit effort="30" velocity="1.0" lower="0.0" upper="1.0" />
     </joint>
-    <!-- Finger 1-->
-    <link name="Finger1">
+    <!-- Gripper Base -->
+    <link name="finger_1_link">
         <collision>
-            <origin rpy="-1.57 0 0" xyz="-0.075 -0.038 0.075" />
+            <origin rpy="0 0 0" xyz="0 0 0" />
             <geometry>
-                <mesh filename="package://fanuc_lrmate200id_support/meshes/gripper/collision/Gripper_finger.STL" scale="0.001 0.001 0.001" />
+                <mesh filename="package://fanuc_lrmate200id_support/meshes/gripper/collision/finger_1.stl" scale="0.001 0.001 0.001" />
             </geometry>
         </collision>
         <visual>
-            <origin rpy="-1.57 0 0" xyz="-0.075 -0.038 0.075" />
+            <origin rpy="0 0 0" xyz="0 0 0" />
             <geometry>
-                <mesh filename="package://fanuc_lrmate200id_support/meshes/gripper/visual/Gripper_finger.STL" scale="0.001 0.001 0.001" />
+                <mesh filename="package://fanuc_lrmate200id_support/meshes/gripper/visual/finger_1.stl" scale="0.001 0.001 0.001" />
             </geometry>
             <material name="">
-                <color rgba="0.278431372549 0.278431372549 0.278431372549 1.0" />
+                <color rgba="0.5 0.5 0.5 1.0" />
             </material>
         </visual>
-<inertial>
+        <inertial>
             <origin rpy="0 0 0" xyz="0.00112 0.04196 0" />
-            <mass value="0.17495" />
-            <inertia ixx="0.002449587" ixy="-0.00141880714" ixz="-0.00044070839" iyy=".00018834795" iyz="-0.00067806067" izz=".00315304482" />
+            <mass value="1.067" />
+            <inertia ixx="0.00372062398" ixy="-0.000013337910" ixz="0.000000013" iyy=".00223540544" iyz="-0.00000003496" izz=".003641916" />
         </inertial>
     </link>
-    <!-- Gripper Base Finger 2 Joint-->
-    <joint name="Gripper_Finger2" type="revolute">
-        <parent link="Gripper_Base" />
-        <child link="Finger2" />
-        <origin rpy="0 0 0" xyz="-0.04448 -0.04 -0.09533" />
-        <axis xyz="0 1 0" />
-        <dynamics damping="0.7" />
-        <limit effort="1" lower="-0.0872" upper="0.0872" velocity="6.1087" />
+    <gazebo reference="finger_1_link">
+        <material>Gazebo/Black</material>
+    </gazebo>
+            <!-- Part 6 Gripper Base Joint -->
+    <joint name="finer_2_to_mid_layer" type="prismatic">
+        <parent link="mid_layer_link" />
+        <child link="finger_2_link" />
+        <origin rpy="0 0 0" xyz="0.10 -0.032 0.0" />
+        <limit effort="30" velocity="1.0" lower="0.0" upper="1.0" />
     </joint>
-    <!-- Finger 2-->
-    <link name="Finger2">
+    <!-- Gripper Base -->
+    <link name="finger_2_link">
         <collision>
-            <origin rpy="-1.57 0 0" xyz="-0.075 -0.038 0.075" />
+            <origin rpy="0 0 0" xyz="0 0 0" />
             <geometry>
-                <mesh filename="package://fanuc_lrmate200id_support/meshes/gripper/collision/Gripper_finger.STL" scale="0.001 0.001 0.001" />
+                <mesh filename="package://fanuc_lrmate200id_support/meshes/gripper/collision/finger_2.stl" scale="0.001 0.001 0.001" />
             </geometry>
         </collision>
         <visual>
-            <origin rpy="-1.57 0 0" xyz="-0.075 -0.038 0.075" />
+            <origin rpy="0 0 0" xyz="0 0 0" />
             <geometry>
-                <mesh filename="package://fanuc_lrmate200id_support/meshes/gripper/visual/Gripper_finger.STL" scale="0.001 0.001 0.001" />
+                <mesh filename="package://fanuc_lrmate200id_support/meshes/gripper/visual/finger_2.stl" scale="0.001 0.001 0.001" />
             </geometry>
             <material name="">
-                <color rgba="0.278431372549 0.278431372549 0.278431372549 1.0" />
+                <color rgba="0.5 0.5 0.5 1.0" />
             </material>
         </visual>
-<inertial>
+        <inertial>
             <origin rpy="0 0 0" xyz="0.00112 0.04196 0" />
-            <mass value="0.17495" />
-            <inertia ixx="0.002449587" ixy="-0.00141880714" ixz="-0.00044070839" iyy=".00018834795" iyz="-0.00067806067" izz=".00315304482" />
+            <mass value="1.067" />
+            <inertia ixx="0.00372062398" ixy="-0.000013337910" ixz="0.000000013" iyy=".00223540544" iyz="-0.00000003496" izz=".003641916" />
         </inertial>
     </link>
-    <transmission name="trans_Part6_Gripper_Base">
-        <type>transmission_interface/SimpleTransmission</type>
-        <joint name="Part6_Gripper_Base">
-            <hardwareInterface>hardware_interface/PositionJointInterface</hardwareInterface>
-        </joint>
-        <actuator name="Part6_Gripper_Base_motor">
-            <hardwareInterface>hardware_interface/PositionJointInterface</hardwareInterface>
-            <mechanicalReduction>1</mechanicalReduction>
-        </actuator>
-    </transmission>
-    <transmission name="trans_Gripper_Finger3">
-        <type>transmission_interface/SimpleTransmission</type>
-        <joint name="Gripper_Finger3">
-            <hardwareInterface>hardware_interface/PositionJointInterface</hardwareInterface>
-        </joint>
-        <actuator name="Gripper_Finger3_motor">
-            <hardwareInterface>hardware_interface/PositionJointInterface</hardwareInterface>
-            <mechanicalReduction>1</mechanicalReduction>
-        </actuator>
-    </transmission>
-    <transmission name="trans_Gripper_Finger1">
-        <type>transmission_interface/SimpleTransmission</type>
-        <joint name="Gripper_Finger1">
-            <hardwareInterface>hardware_interface/PositionJointInterface</hardwareInterface>
-        </joint>
-        <actuator name="Gripper_Finger1_motor">
-            <hardwareInterface>hardware_interface/PositionJointInterface</hardwareInterface>
-            <mechanicalReduction>1</mechanicalReduction>
-        </actuator>
-    </transmission>
-    <transmission name="trans_Gripper_Finger2">
-        <type>transmission_interface/SimpleTransmission</type>
-        <joint name="Gripper_Finger2">
-            <hardwareInterface>hardware_interface/PositionJointInterface</hardwareInterface>
-        </joint>
-        <actuator name="Gripper_Finger2_motor">
-            <hardwareInterface>hardware_interface/PositionJointInterface</hardwareInterface>
-            <mechanicalReduction>1</mechanicalReduction>
-        </actuator>
-    </transmission>
+    <gazebo reference="finger_2_link">
+        <material>Gazebo/Black</material>
+    </gazebo>
 	</xacro:macro>
 </robot>

File: fanuc_lrmate200id_support/urdf/lrmate200id7l.xacro (robot description, xacro)
@@ -2,4 +2,6 @@
 <robot name="fanuc_lrmate200id7l" xmlns:xacro="http://www.ros.org/wiki/xacro">
   <xacro:include filename="$(find fanuc_lrmate200id_support)/urdf/lrmate200id7l_macro.xacro"/>
+  <xacro:include filename="$(find fanuc_lrmate200id_support)/urdf/gripper_macro.xacro"/>
   <xacro:fanuc_lrmate200id7l prefix=""/>
+  <xacro:gripper prefix=""/>
 </robot>

Commit message: update gripper

File: fanuc_lrmate200id_support/urdf/gripper_macro.xacro (robot description, xacro)
@@ -6,5 +6,5 @@
         <parent link="link_6" />
         <child link="gripper_base_link" />
-        <origin rpy="0 0 0" xyz="0.05 0 0.0" />
+        <origin rpy="0 0 0" xyz="0.06 0 0.0" />
     </joint>
     <!-- Gripper Base -->
@@ -67,9 +67,10 @@
     </gazebo>
             <!-- Part 6 Gripper Base Joint -->
-    <joint name="finger_1_to_mid_layer" type="prismatic">
+    <joint name="finger_1_to_mid_layer" type="fixed">
         <parent link="mid_layer_link" />
         <child link="finger_1_link" />
+        <axis xyz="0 1 0" />
         <origin rpy="3.14 0 0" xyz="0.10 0.032 0.0" />
-        <limit effort="30" velocity="1.0" lower="0.0" upper="1.0" />
+        <limit effort="30" velocity="1.0" lower="-0.2" upper="0.2" />
     </joint>
     <!-- Gripper Base -->
@@ -100,9 +101,10 @@
     </gazebo>
             <!-- Part 6 Gripper Base Joint -->
-    <joint name="finer_2_to_mid_layer" type="prismatic">
+    <joint name="finer_2_to_mid_layer" type="fixed">
         <parent link="mid_layer_link" />
         <child link="finger_2_link" />
+        <axis xyz="0 1 0" />
         <origin rpy="0 0 0" xyz="0.10 -0.032 0.0" />
-        <limit effort="30" velocity="1.0" lower="0.0" upper="1.0" />
+        <limit effort="30" velocity="1.0" lower="-0.2" upper="0.2" />
     </joint>
     <!-- Gripper Base -->

Commit message: adjust gripper distance to link6

File: fanuc_lrmate200id_support/urdf/gripper_macro.xacro (robot description, xacro)
@@ -6,5 +6,5 @@
         <parent link="link_6" />
         <child link="gripper_base_link" />
-        <origin rpy="0 0 0" xyz="0.06 0 0.0" />
+        <origin rpy="0 0 0" xyz="0.04 0 0.0" />
     </joint>
     <!-- Gripper Base -->
@@ -71,5 +71,5 @@
         <child link="finger_1_link" />
         <axis xyz="0 1 0" />
-        <origin rpy="3.14 0 0" xyz="0.10 0.032 0.0" />
+        <origin rpy="3.14 0 0" xyz="0.097 0.032 0.0" />
         <limit effort="30" velocity="1.0" lower="-0.2" upper="0.2" />
     </joint>
@@ -105,5 +105,5 @@
         <child link="finger_2_link" />
         <axis xyz="0 1 0" />
-        <origin rpy="0 0 0" xyz="0.10 -0.032 0.0" />
+        <origin rpy="0 0 0" xyz="0.097 -0.032 0.0" />
         <limit effort="30" velocity="1.0" lower="-0.2" upper="0.2" />
     </joint>

File: fanuc_lrmate200id_support/urdf/lrmate200id7l_macro.xacro (robot description, xacro)
@@ -216,17 +216,4 @@
     </joint>
     <link name="${prefix}tool0">
-      <visual>
-        <origin xyz="0 0 0" rpy="0 0 0"/>
-        <geometry>
-          <mesh filename="package://fanuc_lrmate200id_support/meshes/lrmate200id/visual/link_6.stl"/>
-        </geometry>
-        <xacro:material_fanuc_black />
-      </visual>
-      <collision>
-        <origin xyz="0 0 0" rpy="0 0 0"/>
-        <geometry>
-          <mesh filename="package://fanuc_lrmate200id_support/meshes/lrmate200id/collision/link_6.stl"/>
-        </geometry>
-      </collision>
     </link>
     <joint name="${prefix}link_6-tool0" type="fixed">
