Commit message: Camera:: Set it same as real

File: fanuc_lrmate200id_gazebo/urdf/asus_xtion_macro.xacro (robot description, xacro)
@@ -2,11 +2,14 @@
 <robot xmlns:xacro="http://www.ros.org/wiki/xacro">
 <xacro:macro name="asus_xtion" params="prefix">
-    <!-- Part 6 Gripper Base Joint -->
 <joint name="camera_joint" type="fixed">
-    <parent link="base_link" />
+    <parent link="link_4" />
     <child link="camera_link" />
-    <origin rpy="0 1.57 0" xyz="0.6 0.0 1.6" />
+    <origin rpy="-0.0037 1.50600 -0.0031"
+     xyz="0.32273 0.01841 -0.06556" />
     <axis xyz="0 0 0" />
 </joint>
+<gazebo reference="camera_link">
+  <gravity>0</gravity>
+</gazebo>
 <link name="camera_link">
     <collision name="collision">

File: fanuc_lrmate200id_gazebo/urdf/lrmate200id7l.xacro (robot description, xacro)
@@ -6,5 +6,7 @@
 <robot name="fanuc_lrmate200id7l" xmlns:xacro="http://www.ros.org/wiki/xacro">
 <xacro:include filename="$(find fanuc_lrmate200id_gazebo)/urdf/lrmate200id7l_macro.xacro"/>
-  <xacro:fanuc_lrmate200id7l_robot prefix=""/>
+<xacro:include filename="$(find fanuc_lrmate200id_gazebo)/urdf/asus_xtion_macro.xacro"/>
+<xacro:fanuc_lrmate200id7l_robot prefix=""/>
+<xacro:asus_xtion prefix=""/>
   <!-- Fix robot to Gazebo world -->
   <link name="world"/>
