Commit message: add cameras to all arms

File: fanuc_lrmate200id_gazebo/urdf/lrmate200id.xacro (robot description, xacro)
@@ -2,5 +2,9 @@
 <robot name="fanuc_lrmate200id" xmlns:xacro="http://www.ros.org/wiki/xacro">
   <xacro:include filename="$(find fanuc_lrmate200id_gazebo)/urdf/lrmate200id_macro.xacro"/>
+  <xacro:include filename="$(find fanuc_lrmate200id_gazebo)/urdf/_d435.urdf.xacro" />
   <xacro:fanuc_lrmate200id_robot prefix=""/>
+<sensor_d435 parent="link_6">
+  <origin xyz="0.0248461355134 0.0274223973678 0.088426501091" rpy="0 0 0"/>
+</sensor_d435>
   <!-- Fix robot to Gazebo world -->
   <link name="world"/>

File: fanuc_m20ia_gazebo/urdf/m20ia.xacro (robot description, xacro)
@@ -2,5 +2,9 @@
 <robot name="fanuc_m20ia" xmlns:xacro="http://www.ros.org/wiki/xacro">
   <xacro:include filename="$(find fanuc_m20ia_gazebo)/urdf/m20ia_macro.xacro"/>
+  <xacro:include filename="$(find fanuc_m20ia_gazebo)/urdf/_d435.urdf.xacro" />
   <xacro:fanuc_m20ia_robot prefix=""/>
+<sensor_d435 parent="link_6">
+  <origin xyz="0.0248461355134 0.0274223973678 0.088426501091" rpy="0 0 0"/>
+</sensor_d435>
   <!-- Fix robot to Gazebo world -->
   <link name="world"/>

File: fanuc_r2000ic_gazebo/urdf/r2000ic.xacro (robot description, xacro)
@@ -2,5 +2,9 @@
 <robot name="fanuc_r2000ic" xmlns:xacro="http://www.ros.org/wiki/xacro">
   <xacro:include filename="$(find fanuc_r2000ic_gazebo)/urdf/r2000ic_macro.xacro"/>
+  <xacro:include filename="$(find fanuc_r2000ic_gazebo)/urdf/_d435.urdf.xacro" />
   <xacro:fanuc_r2000ic_robot prefix=""/>
+<sensor_d435 parent="link_6">
+  <origin xyz="0.0248461355134 0.0274223973678 0.088426501091" rpy="0 0 0"/>
+</sensor_d435>
   <!-- Fix robot to Gazebo world -->
   <link name="world"/>
