Commit message: make simulation pick place work

File: fanuc_lrmate200id_gazebo/urdf/_d435.urdf.xacro (robot description, xacro)
@@ -15,5 +15,5 @@
     <xacro:property name="d435_cam_depth_to_left_ir_offset" value="0.0"/>
     <xacro:property name="d435_cam_depth_to_right_ir_offset" value="-0.050"/>
-    <xacro:property name="d435_cam_depth_to_color_offset" value="0.015"/>
+    <xacro:property name="d435_cam_depth_to_color_offset" value="0.000"/>
     <!-- The following values model the aluminum peripherial case for the
   	D435 camera, with the camera joint represented by the actual

Commit message: base_in_hand tests

File: fanuc_lrmate200id_gazebo/urdf/_d435.urdf.xacro (robot description, xacro)
@@ -29,5 +29,5 @@
     <xacro:property name="d435_cam_depth_pz" value="${d435_cam_height/2}"/>
     <material name="${name}_aluminum">
-	  <color rgba="0.5 0.5 0.5 1"/>
+	  <color rgba="0.5 0.8 0.5 1"/>
     </material>
     <!-- camera body, with origin at bottom screw mount -->
@@ -39,5 +39,5 @@
     <link name="${name}_bottom_screw_frame"/>
     <joint name="${name}_link_joint" type="fixed">
-      <origin xyz="0 ${d435_cam_depth_py} ${d435_cam_depth_pz}" rpy="0 0 0"/>
+      <origin xyz="0 0 0" rpy="0 0 0"/>
       <parent link="${name}_bottom_screw_frame"/>
       <child link="${name}_link" />

File: fanuc_lrmate200id_gazebo/urdf/lrmate200id7l_base_in_hand_calib.xacro (robot description, xacro)
@@ -11,4 +11,17 @@
   <origin xyz="0.9 0.0 0.6" rpy="0 2.35619 0"/>
 </sensor_d435>
+<link name="aruco_marker_link">
+    <visual>
+      <origin xyz="0 0 0" rpy="0 0 0"/>
+      <geometry>
+        <mesh filename="package://fanuc_lrmate200id_gazebo/meshes/aruco_marker_202_100mm/meshes/aruco_marker_202_100mm.dae"/>
+      </geometry>
+    </visual>
+</link>
+<joint name="marker-link_6-fixed" type="fixed">
+  <parent link="link_6"/>
+  <child link="aruco_marker_link"/>
+  <origin xyz="0.05 0.0 -0.25" rpy="0.0 0.0 0.0" />
+</joint>
   <!-- Fix robot to Gazebo world -->
   <link name="world"/>

Commit message: yet another bug has been treated as it should

File: fanuc_lrmate200id_gazebo/urdf/_d435.urdf.xacro (robot description, xacro)
@@ -15,5 +15,5 @@
     <xacro:property name="d435_cam_depth_to_left_ir_offset" value="0.0"/>
     <xacro:property name="d435_cam_depth_to_right_ir_offset" value="-0.050"/>
-    <xacro:property name="d435_cam_depth_to_color_offset" value="0.000"/>
+    <xacro:property name="d435_cam_depth_to_color_offset" value="0.015"/>
     <!-- The following values model the aluminum peripherial case for the
   	D435 camera, with the camera joint represented by the actual
@@ -29,5 +29,5 @@
     <xacro:property name="d435_cam_depth_pz" value="${d435_cam_height/2}"/>
     <material name="${name}_aluminum">
-	  <color rgba="0.5 0.8 0.5 1"/>
+	  <color rgba="0.5 0.5 0.5 1"/>
     </material>
     <!-- camera body, with origin at bottom screw mount -->
@@ -39,5 +39,5 @@
     <link name="${name}_bottom_screw_frame"/>
     <joint name="${name}_link_joint" type="fixed">
-      <origin xyz="0 0 0" rpy="0 0 0"/>
+      <origin xyz="0 ${d435_cam_depth_py} ${d435_cam_depth_pz}" rpy="0 0 0"/>
       <parent link="${name}_bottom_screw_frame"/>
       <child link="${name}_link" />

Commit message: upstream update for camera urdf

File: fanuc_lrmate200id_gazebo/urdf/_d435.urdf.xacro (robot description, xacro)
@@ -61,5 +61,5 @@
       <inertial>
         <!-- The following are not reliable values, and should not be used for modeling -->
-        <mass value="0.01" />
+        <mass value="0.564" />
         <origin xyz="0 0 0" />
         <inertia ixx="0.003881243" ixy="0.0" ixz="0.0" iyy="0.000498940" iyz="0.0" izz="0.003879257" />
