Commit message: replace kinematics plugin of m20ia

File: fanuc_m20ia_support/urdf/m20ia_macro.xacro (robot description, xacro)
@@ -181,5 +181,5 @@
     </joint>
     <joint name="${prefix}joint_4" type="revolute">
-      <origin xyz="0 0 0.250" rpy="0 0 0"/>
+      <origin xyz="0 0 0.150" rpy="0 0 0"/>
       <parent link="${prefix}link_3"/>
       <child link="${prefix}link_4"/>
@@ -188,5 +188,5 @@
     </joint>
     <joint name="${prefix}joint_5" type="revolute">
-      <origin xyz="0.835 0 0" rpy="0 0 0"/>
+      <origin xyz="0.860 0 0" rpy="0 0 0"/>
       <parent link="${prefix}link_4"/>
       <child link="${prefix}link_5"/>
