Commit message: fix simulated realsense issues

File: fanuc_m20ia_gazebo/urdf/_d435.gazebo.xacro (robot description, xacro)
@@ -9,5 +9,5 @@
     <!-- Load parameters to model's main link-->
     <xacro:property name="deg_to_rad" value="0.01745329251994329577" />
-    <gazebo reference="${reference_link}">
+      <gazebo reference="${reference_link}">
       <turnGravityOff>true</turnGravityOff>
       <self_collide>0</self_collide>
@@ -28,6 +28,6 @@
           <horizontal_fov>${85.2*deg_to_rad}</horizontal_fov>
           <image>
-            <width>640</width>
-            <height>480</height>
+            <width>1280</width>
+            <height>720</height>
             <format>RGB_INT8</format>
           </image>
@@ -50,6 +50,6 @@
           <horizontal_fov>${85.2*deg_to_rad}</horizontal_fov>
           <image>
-            <width>640</width>
-            <height>480</height>
+            <width>1280</width>
+            <height>720</height>
             <format>L_INT8</format>
           </image>
@@ -72,6 +72,6 @@
           <horizontal_fov>${85.2*deg_to_rad}</horizontal_fov>
           <image>
-            <width>640</width>
-            <height>480</height>
+            <width>1280</width>
+            <height>720</height>
             <format>L_INT8</format>
           </image>
@@ -94,6 +94,6 @@
           <horizontal_fov>${85.2*deg_to_rad}</horizontal_fov>
           <image>
-            <width>640</width>
-            <height>480</height>
+            <width>1280</width>
+            <height>720</height>
           </image>
           <clip>

File: fanuc_m20ia_gazebo/urdf/_d435.urdf.xacro (robot description, xacro)
@@ -61,5 +61,5 @@
       <inertial>
         <!-- The following are not reliable values, and should not be used for modeling -->
-        <mass value="0.01" />
+        <mass value="0.564" />
         <origin xyz="0 0 0" />
         <inertia ixx="0.003881243" ixy="0.0" ixz="0.0" iyy="0.000498940" iyz="0.0" izz="0.003879257" />

File: fanuc_r2000ic_gazebo/urdf/_d435.gazebo.xacro (robot description, xacro)
@@ -9,5 +9,5 @@
     <!-- Load parameters to model's main link-->
     <xacro:property name="deg_to_rad" value="0.01745329251994329577" />
-    <gazebo reference="${reference_link}">
+       <gazebo reference="${reference_link}">
       <turnGravityOff>true</turnGravityOff>
       <self_collide>0</self_collide>
@@ -28,6 +28,6 @@
           <horizontal_fov>${85.2*deg_to_rad}</horizontal_fov>
           <image>
-            <width>640</width>
-            <height>480</height>
+            <width>1280</width>
+            <height>720</height>
             <format>RGB_INT8</format>
           </image>
@@ -50,6 +50,6 @@
           <horizontal_fov>${85.2*deg_to_rad}</horizontal_fov>
           <image>
-            <width>640</width>
-            <height>480</height>
+            <width>1280</width>
+            <height>720</height>
             <format>L_INT8</format>
           </image>
@@ -72,6 +72,6 @@
           <horizontal_fov>${85.2*deg_to_rad}</horizontal_fov>
           <image>
-            <width>640</width>
-            <height>480</height>
+            <width>1280</width>
+            <height>720</height>
             <format>L_INT8</format>
           </image>
@@ -94,6 +94,6 @@
           <horizontal_fov>${85.2*deg_to_rad}</horizontal_fov>
           <image>
-            <width>640</width>
-            <height>480</height>
+            <width>1280</width>
+            <height>720</height>
           </image>
           <clip>

File: fanuc_r2000ic_gazebo/urdf/_d435.urdf.xacro (robot description, xacro)
@@ -61,5 +61,5 @@
       <inertial>
         <!-- The following are not reliable values, and should not be used for modeling -->
-        <mass value="0.01" />
+        <mass value="0.564" />
         <origin xyz="0 0 0" />
         <inertia ixx="0.003881243" ixy="0.0" ixz="0.0" iyy="0.000498940" iyz="0.0" izz="0.003879257" />
